Commit message: Implemented the Jetmax arm properly

File: src/main_package/models/jetmax_description/urdf/jetmax.xacro (robot description, xacro)
@@ -92,5 +92,5 @@
 		<visual>
 			<geometry>
-				<mesh filename="package://jetmax_description/meshes/Base.STL" />
+				<mesh filename="package://src/main_package/models/jetmax_description/jetmax_description/meshes/Base.STL" />
 			</geometry>
 			<origin xyz="0 0 0 " rpy="0 0 0" />
@@ -101,5 +101,5 @@
 		<collision>
 			<geometry>
-				<mesh filename="package://jetmax_description/meshes/Base.STL" />
+				<mesh filename="package://src/main_package/models/jetmax_description/jetmax_description/meshes/Base.STL" />
 			</geometry>
 			<origin xyz="0 0 0 " rpy="0 0 0" />
@@ -119,5 +119,5 @@
 			<origin xyz="0 0 0" rpy="0 0 0" />
 			<geometry>
-				<mesh filename="package://jetmax_description/meshes/Link1.STL" />
+				<mesh filename="package://src/main_package/models/jetmax_description/jetmax_description/meshes/Link1.STL" />
 			</geometry>
 			<material name="">
@@ -127,5 +127,5 @@
 		<collision>
 			<geometry>
-				<mesh filename="package://jetmax_description/meshes/Link1.STL" />
+				<mesh filename="package://src/main_package/models/jetmax_description/jetmax_description/meshes/Link1.STL" />
 			</geometry>
 			<origin xyz="0 0 0" rpy="0 0 0" />
@@ -145,5 +145,5 @@
 			<origin xyz="0 0 0" rpy="0 0 0" />
 			<geometry>
-				<mesh filename="package://jetmax_description/meshes/Link2.STL" />
+				<mesh filename="package://src/main_package/models/jetmax_description/jetmax_description/meshes/Link2.STL" />
 			</geometry>
 			<material name="">
@@ -153,5 +153,5 @@
 		<collision>
 			<geometry>
-				<mesh filename="package://jetmax_description/meshes/Link2.STL" />
+				<mesh filename="package://src/main_package/models/jetmax_description/jetmax_description/meshes/Link2.STL" />
 			</geometry>
 			<origin xyz="0 0 0" rpy="0 0 0" />
@@ -171,13 +171,13 @@
 			<origin xyz="0 0 0" rpy="0 0 0" />
 			<geometry>
-				<mesh filename="package://jetmax_description/meshes/Link3.STL" />
-			</geometry>
-			<material name="">
-				<color rgba="0.3 0.3 0.3 1" />
-			</material>
-		</visual>
-		<collision>
-			<geometry>
-				<mesh filename="package://jetmax_description/meshes/Link3.STL" />
+				<mesh filename="package://src/main_package/models/jetmax_description/jetmax_description/meshes/Link3.STL" />
+			</geometry>
+			<material name="">
+				<color rgba="0.3 0.3 0.3 1" />
+			</material>
+		</visual>
+		<collision>
+			<geometry>
+				<mesh filename="package://src/main_package/models/jetmax_description/jetmax_description/meshes/Link3.STL" />
 			</geometry>
 			<origin xyz="0 0 0" rpy="0 0 0" />
@@ -197,14 +197,14 @@
 			<origin xyz="0 0 0" rpy="0 0 0" />
 			<geometry>
-				<mesh filename="package://jetmax_description/meshes/Link4.STL" />
-			</geometry>
-			<material name="">
-				<color rgba="0.3 0.3 0.3 1" />
-			</material>
-		</visual>
-		<collision>
-			<origin xyz="0 0 0" rpy="0 0 0" />
-			<geometry>
-				<mesh filename="package://jetmax_description/meshes/Link4.STL" />
+				<mesh filename="package://src/main_package/models/jetmax_description/jetmax_description/meshes/Link4.STL" />
+			</geometry>
+			<material name="">
+				<color rgba="0.3 0.3 0.3 1" />
+			</material>
+		</visual>
+		<collision>
+			<origin xyz="0 0 0" rpy="0 0 0" />
+			<geometry>
+				<mesh filename="package://src/main_package/models/jetmax_description/jetmax_description/meshes/Link4.STL" />
 			</geometry>
 			<material name="">
@@ -223,14 +223,14 @@
 			<origin xyz="0 0 0" rpy="0 0 0" />
 			<geometry>
-				<mesh filename="package://jetmax_description/meshes/Link5.STL" />
-			</geometry>
-			<material name="">
-				<color rgba="0.3 0.3 0.3 1" />
-			</material>
-		</visual>
-		<collision>
-			<origin xyz="0 0 0" rpy="0 0 0" />
-			<geometry>
-				<mesh filename="package://jetmax_description/meshes/Link5.STL" />
+				<mesh filename="package://src/main_package/models/jetmax_description/jetmax_description/meshes/Link5.STL" />
+			</geometry>
+			<material name="">
+				<color rgba="0.3 0.3 0.3 1" />
+			</material>
+		</visual>
+		<collision>
+			<origin xyz="0 0 0" rpy="0 0 0" />
+			<geometry>
+				<mesh filename="package://src/main_package/models/jetmax_description/jetmax_description/meshes/Link5.STL" />
 			</geometry>
 			<material name="">
@@ -249,14 +249,14 @@
 			<origin xyz="0 0 0" rpy="0 0 0" />
 			<geometry>
-				<mesh filename="package://jetmax_description/meshes/Link6.STL" />
-			</geometry>
-			<material name="">
-				<color rgba="0.3 0.3 0.3 1" />
-			</material>
-		</visual>
-		<collision>
-			<origin xyz="0 0 0" rpy="0 0 0" />
-			<geometry>
-				<mesh filename="package://jetmax_description/meshes/Link6.STL" />
+				<mesh filename="package://src/main_package/models/jetmax_description/jetmax_description/meshes/Link6.STL" />
+			</geometry>
+			<material name="">
+				<color rgba="0.3 0.3 0.3 1" />
+			</material>
+		</visual>
+		<collision>
+			<origin xyz="0 0 0" rpy="0 0 0" />
+			<geometry>
+				<mesh filename="package://src/main_package/models/jetmax_description/jetmax_description/meshes/Link6.STL" />
 			</geometry>
 			<material name="">
@@ -275,14 +275,14 @@
 			<origin xyz="0 0 0" rpy="0 0 0" />
 			<geometry>
-				<mesh filename="package://jetmax_description/meshes/Link7.STL" />
-			</geometry>
-			<material name="">
-				<color rgba="0.3 0.3 0.3 1" />
-			</material>
-		</visual>
-		<collision>
-			<origin xyz="0 0 0" rpy="0 0 0" />
-			<geometry>
-				<mesh filename="package://jetmax_description/meshes/Link7.STL" />
+				<mesh filename="package://src/main_package/models/jetmax_description/jetmax_description/meshes/Link7.STL" />
+			</geometry>
+			<material name="">
+				<color rgba="0.3 0.3 0.3 1" />
+			</material>
+		</visual>
+		<collision>
+			<origin xyz="0 0 0" rpy="0 0 0" />
+			<geometry>
+				<mesh filename="package://src/main_package/models/jetmax_description/jetmax_description/meshes/Link7.STL" />
 			</geometry>
 			<material name="">
@@ -301,5 +301,5 @@
 			<origin xyz="0 0 0" rpy="0 0 0" />
 			<geometry>
-				<mesh filename="package://jetmax_description/meshes/Suction.STL" />
+				<mesh filename="package://src/main_package/models/jetmax_description/jetmax_description/meshes/Suction.STL" />
 			</geometry>
 			<material name="">
@@ -328,14 +328,14 @@
 			<origin xyz="0 0 0" rpy="0 0 0" />
 			<geometry>
-				<mesh filename="package://jetmax_description/meshes/Link9.STL" />
-			</geometry>
-			<material name="">
-				<color rgba="0.3 0.3 0.3 1" />
-			</material>
-		</visual>
-		<collision>
-			<origin xyz="0 0 0" rpy="0 0 0" />
-			<geometry>
-				<mesh filename="package://jetmax_description/meshes/Link9.STL" />
+				<mesh filename="package://src/main_package/models/jetmax_description/jetmax_description/meshes/Link9.STL" />
+			</geometry>
+			<material name="">
+				<color rgba="0.3 0.3 0.3 1" />
+			</material>
+		</visual>
+		<collision>
+			<origin xyz="0 0 0" rpy="0 0 0" />
+			<geometry>
+				<mesh filename="package://src/main_package/models/jetmax_description/jetmax_description/meshes/Link9.STL" />
 			</geometry>
 			<material name="">
