Commit message: Worked on the Jetmax model

File: src/jetmax_description/urdf/jetmax.xacro (robot description, xacro)
@@ -11,77 +11,4 @@
 		<child link="Base" />
 	</joint>
-	<!-- Bitxh ass joints - dont delete from here. MOdel wont work without it-->
-	<joint name="Joint1" type="revolute">
-        <axis xyz="0 0 1" />
-        <limit effort="10" lower="-3" upper="3" velocity="0.0" />
-        <parent link="Base" />
-        <child link="Link1" />
-        <origin xyz="0 0 0.064273" rpy=" 0 0 0" />
-    </joint>
-    <joint name="Joint2" type="revolute">
-        <axis xyz="-1 0 0" />
-        <limit effort="10" lower="-3" upper="3" velocity="0.0" />
-        <parent link="Link1" />
-        <child link="Link2" />
-        <origin xyz="-0.0041395 -0.0081353 0.021592" rpy="0 0 0" />
-    </joint>
-    <joint name="Joint3" type="revolute">
-        <axis xyz="1 0 0" />
-        <parent link="Link2" />
-        <child link="Link3" />
-        <limit effort="10" lower="-1.45" upper="1.45" velocity="0.0" />
-        <origin xyz="-0.0033882 0 0.12845" rpy="-0.0011788 0 0" />
-    </joint>
-    <joint name="Joint4" type="revolute">
-        <axis xyz="1 0 0" />
-        <limit effort="10" lower="-3" upper="3" velocity="0.0" />
-        <parent link="Link2" />
-        <child link="Link4" />
-        <origin xyz="0.032307 5.2901E-05 0.12853" rpy="0 0 0" />
-    </joint>
-    <joint name="Joint5" type="revolute">
-        <axis xyz="-1 0 0" />
-        <limit effort="10" lower="-3" upper="3" velocity="0.0" />
-        <parent link="Link1" />
-        <child link="Link5" />
-        <origin xyz="0.018067 0.026256 0.045902" rpy="0 0 0" />
-    </joint>
-    <joint name="Joint6" type="revolute">
-        <axis xyz="-1 0 0" />
-        <limit effort="10" lower="-3" upper="3" velocity="0.0" />
-        <parent link="Link1" />
-        <child link="Link6" />
-        <origin xyz="-0.0060277 -0.0081353 0.021592" rpy="0 0 0" />
-    </joint>
-    <joint name="Joint7" type="revolute">
-        <axis xyz="-1 0 0" />
-        <limit effort="10" lower="-3" upper="3" velocity="0.0" />
-        <parent link="Link6" />
-        <child link="Link7" />
-        <origin xyz="0 0.0432 0" rpy="0 0 0" />
-    </joint>
-    <joint name="Joint8" type="revolute">
-        <axis xyz="1 0 0" />
-        <limit effort="10" lower="-3" upper="3" velocity="0.0" />
-        <parent link="Link3" />
-        <child link="Link8" />
-        <origin xyz="0 -0.138 -0.00016405" rpy="0.0011788 0 0" />
-    </joint>
-    <joint name="Joint9" type="revolute">
-        <axis xyz="-1 0 0" />
-        <limit effort="10" lower="-3" upper="3" velocity="0.0" />
-        <parent link="Link8" />
-        <child link="Link9" />
-        <origin xyz="0.031695 -0.034122 0.024493" rpy="0 0 0" />
-    </joint>
-    <!-- virtual joints needed for vacuum_gripper plugin -->
-    <joint name="virtual_end_joint" type="revolute">
-        <axis xyz="0 0 1" />
-        <parent link="Link8" />
-        <child link="virtual_end_effector" />
-        <origin xyz="0.01 -0.017 -0.075" rpy=" 0 0 0" />
-        <limit effort="1" lower="0" upper="0" velocity="0.0" />
-    </joint>
-	<!--  End of bitxh asss joints -->
 	<link name="Base">
 		<inertial>
@@ -92,5 +19,5 @@
 		<visual>
 			<geometry>
-				<mesh filename="package://src/main_package/models/jetmax_description/jetmax_description/meshes/Base.STL" />
+				<mesh filename="package://jetmax_description/meshes/Base.STL" />
 			</geometry>
 			<origin xyz="0 0 0 " rpy="0 0 0" />
@@ -101,5 +28,5 @@
 		<collision>
 			<geometry>
-				<mesh filename="package://src/main_package/models/jetmax_description/jetmax_description/meshes/Base.STL" />
+				<mesh filename="package://jetmax_description/meshes/Base.STL" />
 			</geometry>
 			<origin xyz="0 0 0 " rpy="0 0 0" />
@@ -119,13 +46,13 @@
 			<origin xyz="0 0 0" rpy="0 0 0" />
 			<geometry>
-				<mesh filename="package://src/main_package/models/jetmax_description/jetmax_description/meshes/Link1.STL" />
-			</geometry>
-			<material name="">
-				<color rgba="0.3 0.8 0.3 1" />
-			</material>
-		</visual>
-		<collision>
-			<geometry>
-				<mesh filename="package://src/main_package/models/jetmax_description/jetmax_description/meshes/Link1.STL" />
+				<mesh filename="package://jetmax_description/meshes/Link1.STL" />
+			</geometry>
+			<material name="">
+				<color rgba="0.3 0.8 0.3 1" />
+			</material>
+		</visual>
+		<collision>
+			<geometry>
+				<mesh filename="package://jetmax_description/meshes/Link1.STL" />
 			</geometry>
 			<origin xyz="0 0 0" rpy="0 0 0" />
@@ -145,13 +72,13 @@
 			<origin xyz="0 0 0" rpy="0 0 0" />
 			<geometry>
-				<mesh filename="package://src/main_package/models/jetmax_description/jetmax_description/meshes/Link2.STL" />
-			</geometry>
-			<material name="">
-				<color rgba="0.3 0.8 0.3 1" />
-			</material>
-		</visual>
-		<collision>
-			<geometry>
-				<mesh filename="package://src/main_package/models/jetmax_description/jetmax_description/meshes/Link2.STL" />
+				<mesh filename="package://jetmax_description/meshes/Link2.STL" />
+			</geometry>
+			<material name="">
+				<color rgba="0.3 0.8 0.3 1" />
+			</material>
+		</visual>
+		<collision>
+			<geometry>
+				<mesh filename="package://jetmax_description/meshes/Link2.STL" />
 			</geometry>
 			<origin xyz="0 0 0" rpy="0 0 0" />
@@ -171,13 +98,13 @@
 			<origin xyz="0 0 0" rpy="0 0 0" />
 			<geometry>
-				<mesh filename="package://src/main_package/models/jetmax_description/jetmax_description/meshes/Link3.STL" />
-			</geometry>
-			<material name="">
-				<color rgba="0.3 0.3 0.3 1" />
-			</material>
-		</visual>
-		<collision>
-			<geometry>
-				<mesh filename="package://src/main_package/models/jetmax_description/jetmax_description/meshes/Link3.STL" />
+				<mesh filename="package://jetmax_description/meshes/Link3.STL" />
+			</geometry>
+			<material name="">
+				<color rgba="0.3 0.3 0.3 1" />
+			</material>
+		</visual>
+		<collision>
+			<geometry>
+				<mesh filename="package://jetmax_description/meshes/Link3.STL" />
 			</geometry>
 			<origin xyz="0 0 0" rpy="0 0 0" />
@@ -197,14 +124,14 @@
 			<origin xyz="0 0 0" rpy="0 0 0" />
 			<geometry>
-				<mesh filename="package://src/main_package/models/jetmax_description/jetmax_description/meshes/Link4.STL" />
-			</geometry>
-			<material name="">
-				<color rgba="0.3 0.3 0.3 1" />
-			</material>
-		</visual>
-		<collision>
-			<origin xyz="0 0 0" rpy="0 0 0" />
-			<geometry>
-				<mesh filename="package://src/main_package/models/jetmax_description/jetmax_description/meshes/Link4.STL" />
+				<mesh filename="package://jetmax_description/meshes/Link4.STL" />
+			</geometry>
+			<material name="">
+				<color rgba="0.3 0.3 0.3 1" />
+			</material>
+		</visual>
+		<collision>
+			<origin xyz="0 0 0" rpy="0 0 0" />
+			<geometry>
+				<mesh filename="package://jetmax_description/meshes/Link4.STL" />
 			</geometry>
 			<material name="">
@@ -223,14 +150,14 @@
 			<origin xyz="0 0 0" rpy="0 0 0" />
 			<geometry>
-				<mesh filename="package://src/main_package/models/jetmax_description/jetmax_description/meshes/Link5.STL" />
-			</geometry>
-			<material name="">
-				<color rgba="0.3 0.3 0.3 1" />
-			</material>
-		</visual>
-		<collision>
-			<origin xyz="0 0 0" rpy="0 0 0" />
-			<geometry>
-				<mesh filename="package://src/main_package/models/jetmax_description/jetmax_description/meshes/Link5.STL" />
+				<mesh filename="package://jetmax_description/meshes/Link5.STL" />
+			</geometry>
+			<material name="">
+				<color rgba="0.3 0.3 0.3 1" />
+			</material>
+		</visual>
+		<collision>
+			<origin xyz="0 0 0" rpy="0 0 0" />
+			<geometry>
+				<mesh filename="package://jetmax_description/meshes/Link5.STL" />
 			</geometry>
 			<material name="">
@@ -249,14 +176,14 @@
 			<origin xyz="0 0 0" rpy="0 0 0" />
 			<geometry>
-				<mesh filename="package://src/main_package/models/jetmax_description/jetmax_description/meshes/Link6.STL" />
-			</geometry>
-			<material name="">
-				<color rgba="0.3 0.3 0.3 1" />
-			</material>
-		</visual>
-		<collision>
-			<origin xyz="0 0 0" rpy="0 0 0" />
-			<geometry>
-				<mesh filename="package://src/main_package/models/jetmax_description/jetmax_description/meshes/Link6.STL" />
+				<mesh filename="package://jetmax_description/meshes/Link6.STL" />
+			</geometry>
+			<material name="">
+				<color rgba="0.3 0.3 0.3 1" />
+			</material>
+		</visual>
+		<collision>
+			<origin xyz="0 0 0" rpy="0 0 0" />
+			<geometry>
+				<mesh filename="package://jetmax_description/meshes/Link6.STL" />
 			</geometry>
 			<material name="">
@@ -275,14 +202,14 @@
 			<origin xyz="0 0 0" rpy="0 0 0" />
 			<geometry>
-				<mesh filename="package://src/main_package/models/jetmax_description/jetmax_description/meshes/Link7.STL" />
-			</geometry>
-			<material name="">
-				<color rgba="0.3 0.3 0.3 1" />
-			</material>
-		</visual>
-		<collision>
-			<origin xyz="0 0 0" rpy="0 0 0" />
-			<geometry>
-				<mesh filename="package://src/main_package/models/jetmax_description/jetmax_description/meshes/Link7.STL" />
+				<mesh filename="package://jetmax_description/meshes/Link7.STL" />
+			</geometry>
+			<material name="">
+				<color rgba="0.3 0.3 0.3 1" />
+			</material>
+		</visual>
+		<collision>
+			<origin xyz="0 0 0" rpy="0 0 0" />
+			<geometry>
+				<mesh filename="package://jetmax_description/meshes/Link7.STL" />
 			</geometry>
 			<material name="">
@@ -301,5 +228,5 @@
 			<origin xyz="0 0 0" rpy="0 0 0" />
 			<geometry>
-				<mesh filename="package://src/main_package/models/jetmax_description/jetmax_description/meshes/Suction.STL" />
+				<mesh filename="package://jetmax_description/meshes/Suction.STL" />
 			</geometry>
 			<material name="">
@@ -328,14 +255,14 @@
 			<origin xyz="0 0 0" rpy="0 0 0" />
 			<geometry>
-				<mesh filename="package://src/main_package/models/jetmax_description/jetmax_description/meshes/Link9.STL" />
-			</geometry>
-			<material name="">
-				<color rgba="0.3 0.3 0.3 1" />
-			</material>
-		</visual>
-		<collision>
-			<origin xyz="0 0 0" rpy="0 0 0" />
-			<geometry>
-				<mesh filename="package://src/main_package/models/jetmax_description/jetmax_description/meshes/Link9.STL" />
+				<mesh filename="package://jetmax_description/meshes/Link9.STL" />
+			</geometry>
+			<material name="">
+				<color rgba="0.3 0.3 0.3 1" />
+			</material>
+		</visual>
+		<collision>
+			<origin xyz="0 0 0" rpy="0 0 0" />
+			<geometry>
+				<mesh filename="package://jetmax_description/meshes/Link9.STL" />
 			</geometry>
 			<material name="">

Commit message: Loading Jetmax robot (joints not working)
Co-authored-by: Erik Lindby <ELindby@users.noreply.github.com>

File: src/jetmax_description/urdf/jetmax.xacro (robot description, xacro)
@@ -6,4 +6,5 @@
 	<!-- Used for fixing robot to Gazebo 'base_link' -->
 	<link name="world" />
+	<!-- Creates root link -->
 	<joint name="base_joint" type="fixed">
 		<origin xyz="0 0 0" rpy="0 0 0" />
@@ -19,5 +20,7 @@
 		<visual>
 			<geometry>
-				<mesh filename="package://jetmax_description/meshes/Base.STL" />
+				<!-- <mesh filename="$package://jetmax_description/meshes/Base.STL" /> -->
+				<mesh filename="$(find jetmax_description)/meshes/Base.STL"/>
+				<!-- ${find toycar}/meshes/wheel.stl -->
 			</geometry>
 			<origin xyz="0 0 0 " rpy="0 0 0" />
@@ -28,5 +31,5 @@
 		<collision>
 			<geometry>
-				<mesh filename="package://jetmax_description/meshes/Base.STL" />
+				<mesh filename="$(find jetmax_description)/meshes/Base.STL" />
 			</geometry>
 			<origin xyz="0 0 0 " rpy="0 0 0" />
@@ -46,13 +49,13 @@
 			<origin xyz="0 0 0" rpy="0 0 0" />
 			<geometry>
-				<mesh filename="package://jetmax_description/meshes/Link1.STL" />
-			</geometry>
-			<material name="">
-				<color rgba="0.3 0.8 0.3 1" />
-			</material>
-		</visual>
-		<collision>
-			<geometry>
-				<mesh filename="package://jetmax_description/meshes/Link1.STL" />
+				<mesh filename="$(find jetmax_description)/meshes/Link1.STL" />
+			</geometry>
+			<material name="">
+				<color rgba="0.3 0.8 0.3 1" />
+			</material>
+		</visual>
+		<collision>
+			<geometry>
+				<mesh filename="$(find jetmax_description)/meshes/Link1.STL" />
 			</geometry>
 			<origin xyz="0 0 0" rpy="0 0 0" />
@@ -72,13 +75,13 @@
 			<origin xyz="0 0 0" rpy="0 0 0" />
 			<geometry>
-				<mesh filename="package://jetmax_description/meshes/Link2.STL" />
-			</geometry>
-			<material name="">
-				<color rgba="0.3 0.8 0.3 1" />
-			</material>
-		</visual>
-		<collision>
-			<geometry>
-				<mesh filename="package://jetmax_description/meshes/Link2.STL" />
+				<mesh filename="$(find jetmax_description)/meshes/Link2.STL" />
+			</geometry>
+			<material name="">
+				<color rgba="0.3 0.8 0.3 1" />
+			</material>
+		</visual>
+		<collision>
+			<geometry>
+				<mesh filename="$(find jetmax_description)/meshes/Link2.STL" />
 			</geometry>
 			<origin xyz="0 0 0" rpy="0 0 0" />
@@ -98,13 +101,13 @@
 			<origin xyz="0 0 0" rpy="0 0 0" />
 			<geometry>
-				<mesh filename="package://jetmax_description/meshes/Link3.STL" />
-			</geometry>
-			<material name="">
-				<color rgba="0.3 0.3 0.3 1" />
-			</material>
-		</visual>
-		<collision>
-			<geometry>
-				<mesh filename="package://jetmax_description/meshes/Link3.STL" />
+				<mesh filename="$(find jetmax_description)/meshes/Link3.STL" />
+			</geometry>
+			<material name="">
+				<color rgba="0.3 0.3 0.3 1" />
+			</material>
+		</visual>
+		<collision>
+			<geometry>
+				<mesh filename="$(find jetmax_description)/meshes/Link3.STL" />
 			</geometry>
 			<origin xyz="0 0 0" rpy="0 0 0" />
@@ -124,14 +127,14 @@
 			<origin xyz="0 0 0" rpy="0 0 0" />
 			<geometry>
-				<mesh filename="package://jetmax_description/meshes/Link4.STL" />
-			</geometry>
-			<material name="">
-				<color rgba="0.3 0.3 0.3 1" />
-			</material>
-		</visual>
-		<collision>
-			<origin xyz="0 0 0" rpy="0 0 0" />
-			<geometry>
-				<mesh filename="package://jetmax_description/meshes/Link4.STL" />
+				<mesh filename="$(find jetmax_description)/meshes/Link4.STL" />
+			</geometry>
+			<material name="">
+				<color rgba="0.3 0.3 0.3 1" />
+			</material>
+		</visual>
+		<collision>
+			<origin xyz="0 0 0" rpy="0 0 0" />
+			<geometry>
+				<mesh filename="$(find jetmax_description)/meshes/Link4.STL" />
 			</geometry>
 			<material name="">
@@ -150,14 +153,14 @@
 			<origin xyz="0 0 0" rpy="0 0 0" />
 			<geometry>
-				<mesh filename="package://jetmax_description/meshes/Link5.STL" />
-			</geometry>
-			<material name="">
-				<color rgba="0.3 0.3 0.3 1" />
-			</material>
-		</visual>
-		<collision>
-			<origin xyz="0 0 0" rpy="0 0 0" />
-			<geometry>
-				<mesh filename="package://jetmax_description/meshes/Link5.STL" />
+				<mesh filename="$(find jetmax_description)/meshes/Link5.STL" />
+			</geometry>
+			<material name="">
+				<color rgba="0.3 0.3 0.3 1" />
+			</material>
+		</visual>
+		<collision>
+			<origin xyz="0 0 0" rpy="0 0 0" />
+			<geometry>
+				<mesh filename="$(find jetmax_description)/meshes/Link5.STL" />
 			</geometry>
 			<material name="">
@@ -176,14 +179,14 @@
 			<origin xyz="0 0 0" rpy="0 0 0" />
 			<geometry>
-				<mesh filename="package://jetmax_description/meshes/Link6.STL" />
-			</geometry>
-			<material name="">
-				<color rgba="0.3 0.3 0.3 1" />
-			</material>
-		</visual>
-		<collision>
-			<origin xyz="0 0 0" rpy="0 0 0" />
-			<geometry>
-				<mesh filename="package://jetmax_description/meshes/Link6.STL" />
+				<mesh filename="$(find jetmax_description)/meshes/Link6.STL" />
+			</geometry>
+			<material name="">
+				<color rgba="0.3 0.3 0.3 1" />
+			</material>
+		</visual>
+		<collision>
+			<origin xyz="0 0 0" rpy="0 0 0" />
+			<geometry>
+				<mesh filename="$(find jetmax_description)/meshes/Link6.STL" />
 			</geometry>
 			<material name="">
@@ -202,14 +205,14 @@
 			<origin xyz="0 0 0" rpy="0 0 0" />
 			<geometry>
-				<mesh filename="package://jetmax_description/meshes/Link7.STL" />
-			</geometry>
-			<material name="">
-				<color rgba="0.3 0.3 0.3 1" />
-			</material>
-		</visual>
-		<collision>
-			<origin xyz="0 0 0" rpy="0 0 0" />
-			<geometry>
-				<mesh filename="package://jetmax_description/meshes/Link7.STL" />
+				<mesh filename="$(find jetmax_description)/meshes/Link7.STL" />
+			</geometry>
+			<material name="">
+				<color rgba="0.3 0.3 0.3 1" />
+			</material>
+		</visual>
+		<collision>
+			<origin xyz="0 0 0" rpy="0 0 0" />
+			<geometry>
+				<mesh filename="$(find jetmax_description)/meshes/Link7.STL" />
 			</geometry>
 			<material name="">
@@ -228,5 +231,5 @@
 			<origin xyz="0 0 0" rpy="0 0 0" />
 			<geometry>
-				<mesh filename="package://jetmax_description/meshes/Suction.STL" />
+				<mesh filename="$(find jetmax_description)/meshes/Suction.STL" />
 			</geometry>
 			<material name="">
@@ -238,5 +241,5 @@
 		  <origin xyz="0 0 0" rpy="0 0 0" />
 		  <geometry>
-			<mesh filename="package://jetmax_description/meshes/Link8.STL" />
+			<mesh filename="$(find jetmax_description)/meshes/Link8.STL" />
 		  </geometry>
 			<material name="">
@@ -255,14 +258,14 @@
 			<origin xyz="0 0 0" rpy="0 0 0" />
 			<geometry>
-				<mesh filename="package://jetmax_description/meshes/Link9.STL" />
-			</geometry>
-			<material name="">
-				<color rgba="0.3 0.3 0.3 1" />
-			</material>
-		</visual>
-		<collision>
-			<origin xyz="0 0 0" rpy="0 0 0" />
-			<geometry>
-				<mesh filename="package://jetmax_description/meshes/Link9.STL" />
+				<mesh filename="$(find jetmax_description)/meshes/Link9.STL" />
+			</geometry>
+			<material name="">
+				<color rgba="0.3 0.3 0.3 1" />
+			</material>
+		</visual>
+		<collision>
+			<origin xyz="0 0 0" rpy="0 0 0" />
+			<geometry>
+				<mesh filename="$(find jetmax_description)/meshes/Link9.STL" />
 			</geometry>
 			<material name="">

Commit message: Started work on controller for Jetmax

File: src/jetmax_description/urdf/jetmax.xacro (robot description, xacro)
@@ -4,4 +4,27 @@
 	<xacro:include filename="$(find jetmax_description)/urdf/jetmax_joints.xml" />
 	<xacro:include filename="$(find jetmax_description)/urdf/jetmax_trans.xml" />
+	<!-- Test of ros2 control plugin -->
+	<ros2_control name="RRBotSystemPositionOnly" type="system">
+		<hardware>
+		  <plugin>ros2_control_demo_hardware/RRBotSystemPositionOnlyHardware</plugin>
+		  <param name="example_param_hw_start_duration_sec">2.0</param>
+		  <param name="example_param_hw_stop_duration_sec">3.0</param>
+		  <param name="example_param_hw_slowdown">2.0</param>
+		</hardware>
+		<joint name="Joint1">
+		  <command_interface name="position">
+			<param name="min">-1</param>
+			<param name="max">1</param>
+		  </command_interface>
+		  <state_interface name="position"/>
+		</joint>
+		<joint name="Joint2">
+		  <command_interface name="position">
+			<param name="min">-1</param>
+			<param name="max">1</param>
+		  </command_interface>
+		  <state_interface name="position"/>
+		</joint>
+	  </ros2_control>
 	<!-- Used for fixing robot to Gazebo 'base_link' -->
 	<link name="world" />
@@ -12,4 +35,12 @@
 		<child link="Base" />
 	</joint>
+	<!-- <gazebo>
+		<plugin name="gazebo_ros_control" filename="libgazebo_ros_control.so">
+			<robotNamespace>/jetmax</robotNamespace>
+		</plugin>
+	</gazebo> -->
+	<hardware>
+      <plugin>gazebo_ros2_control/GazeboSystem</plugin>
+  	</hardware>
 	<link name="Base">
 		<inertial>

Commit message: Worked on the controller manager, it kinda works
Co-authored-by: jajep18 <jajep18@users.noreply.github.com>

File: src/jetmax_description/urdf/jetmax.xacro (robot description, xacro)
@@ -4,27 +4,4 @@
 	<xacro:include filename="$(find jetmax_description)/urdf/jetmax_joints.xml" />
 	<xacro:include filename="$(find jetmax_description)/urdf/jetmax_trans.xml" />
-	<!-- Test of ros2 control plugin -->
-	<ros2_control name="RRBotSystemPositionOnly" type="system">
-		<hardware>
-		  <plugin>ros2_control_demo_hardware/RRBotSystemPositionOnlyHardware</plugin>
-		  <param name="example_param_hw_start_duration_sec">2.0</param>
-		  <param name="example_param_hw_stop_duration_sec">3.0</param>
-		  <param name="example_param_hw_slowdown">2.0</param>
-		</hardware>
-		<joint name="Joint1">
-		  <command_interface name="position">
-			<param name="min">-1</param>
-			<param name="max">1</param>
-		  </command_interface>
-		  <state_interface name="position"/>
-		</joint>
-		<joint name="Joint2">
-		  <command_interface name="position">
-			<param name="min">-1</param>
-			<param name="max">1</param>
-		  </command_interface>
-		  <state_interface name="position"/>
-		</joint>
-	  </ros2_control>
 	<!-- Used for fixing robot to Gazebo 'base_link' -->
 	<link name="world" />
